Commit message: claude save

File: urdf/Group6Bot_1.urdf (robot description, URDF)
Before this commit: robot com760Bot, 6 links, 5 joints
Joints:
- joint camera_joint: origin xyz=0.25 0 0 rpy=0 0 0 -> xyz=0.0 0 0.35 rpy=0 0.6 0

File: urdf/group6bot_0.urdf.xacro (robot description, xacro)
@@ -132,6 +132,6 @@
   <gazebo reference="base_scan">
     <sensor type="ray" name="laser">
-      <visualize>true</visualize> <ray>
-        <scan><horizontal><samples>360</samples><min_angle>-3.14</min_angle><max_angle>3.14</max_angle></horizontal></scan>
+      <visualize>false</visualize> <ray>
+        <scan><horizontal><samples>360</samples><min_angle>-3.1</min_angle><max_angle>3.1</max_angle></horizontal></scan>
 <!-- This enables the LiDar sensor to have full 360 scan, it is suitable for SLAM and obstacle avoidance. -->
         <range><min>0.15</min><max>12.0</max></range><!-- Reasonable hybrid range for indoor/outdoor. -->
@@ -145,5 +145,5 @@
   <gazebo reference="camera_link">
     <sensor type="camera" name="main_camera">
-<!-- The ROS camera plugin, the topic naming is clean and the frame is assigned correctly. However it has no resolution or FOV specified only the defaults have been used. -->
+      <visualize>false</visualize>
       <plugin name="camera_controller" filename="libgazebo_ros_camera.so">
         <robotNamespace>/group6bot_0</robotNamespace>
