Commit message: bug 2 and RL

File: urdf/Group6Bot_0.urdf.xacro (robot description, xacro)
@@ -173,5 +173,5 @@
     <xacro:cylinder_inertia m="0.1" r="0.05" h="0.05"/>
   </link>
-  <joint name="scan_joint" type="fixed">
+  <joint name="${prefix}/scan_joint" type="fixed">
     <parent link="${prefix}/base_link"/>
     <child link="${prefix}/base_scan"/>
@@ -190,5 +190,5 @@
     <xacro:box_inertia m="0.1" w="0.05" h="0.05" d="0.05"/>
   </link>
-  <joint name="camera_joint" type="fixed">
+  <joint name="${prefix}/camera_joint" type="fixed">
     <parent link="${prefix}/base_link"/>
     <child link="${prefix}/camera_link"/>

File: urdf/Group6Bot_1.urdf.xacro (robot description, xacro)
@@ -147,5 +147,5 @@
         <robotBaseFrame>${robot_name}/base_link</robotBaseFrame>
         <!-- Set to true to publish transforms for the wheel links, defaults to false -->
-        <publishWheelTF>true</publishWheelTF>
+        <publishWheelTF>false</publishWheelTF>
         <!-- Set to true to publish sensor_msgs/JointState on /joint_states for the wheel joints, defaults to false -->
         <publishWheelJointState>true</publishWheelJointState>
